File: board/BLDC_4.kicad_pcb (KiCad board)
At the start: 4 copper layers, 38.5 x 65 mm, 127 parts, among them K1 SERVO, P1 HALL/Encoder, P101 CANBUS, P2 SWD, P3 PWR_COMM, P4 IN+, P5 IN-, P6 MOTOR1, P7 MOTOR2, P9 MOTOR3, Q1 IRFS7530, Q2 IRFS7530, Q3 IRFS7530, Q4 IRFS7530, Q5 IRFS7530, Q6 IRFS7530, U1 STM32F40X_LQFP64, U2 TC2117, U3 DRV8302, U401 SN65HVD232, X1 MINI-USB-SHIELD-32005-201, X2 8MHz 10ppm

Commit message: - implemented complementary transistor package - started layout
Parts:
- removed 1PIN (x2): P***, 1pin
- removed 1PIN (x2): P***, Connect:1pin
- removed C15, C38: 15p, CRF1:SMD-0603_c
- removed C16, C17, C18, C20, C23, C24, C26, C31, C35, C401, C52: 2.2u, CRF1:SMD-0603_c
- removed C19: 120p, CRF1:SMD-0603_c
- removed C21: 6.8n, CRF1:SMD-0603_c
- removed C22: 22n, CRF1:SMD-0603_c
- removed C25, C33: 100u, w_smd_cap:c_tant_B
- removed C27, C32: 100n, CRF1:SMD-0603_c
- removed C28, C29, C30: 220n, CRF1:SMD-0603_c
- removed C34, C36: 2.2n, CRF1:SMD-0603_c
- removed C37: 15u,100V, w_smd_cap:c_2220
- removed C39, C40, C43, C44, C49: 10u,50V, CRF1:SMD-1206
- removed C51: 15u, 100v, w_smd_cap:c_2220
- removed D4: DIODESCH, Diodes_SMD:SMA_Handsoldering
- removed D5: TVS 5V, w_smd_diode:do214ac
- removed G***: oshw_silkscreen-back_3mm, oshw_silkscreen-back_3mm
- removed K1: SERVO, CRF1:pinhead-1X03
- removed L1: 22u, w_smd_inductors:inductor_smd_8x5mm
- removed P101: CANBUS, JST conn:b4b-ph-kl
- removed P2: SWD, CRF1:MICRO_JST_6
- removed P3: PWR_COMM, CRF1:b7b-ph-kl
- removed R103, R104: 22R, CRF1:SMD-0603_r
- removed R401: NI, CRF1:SMD-0603_r
- removed R402: 10k, CRF1:SMD-0603_r
- removed R42, R43: 4R7, CRF1:SMD-0603_r
- removed R46: 39k, CRF1:SMD-0603_r
- removed R48, R49, R50, R51: 100R, CRF1:SMD-0603_r
- removed R53, R54: SHUNT, CRF1:WSLP2726
- removed U401: SN65HVD232, CRF1:SOIC-8-W
- removed X1: MINI-USB-SHIELD-32005-201, CRF1:USB-UX60R-MB-5ST
- removed X2: 8MHz 10ppm, CRF1:Crystal_5x3mm
- added IC1: ACS758, alexmod:CB-PFF, F.Cu at (230.0, 122.0)
- added IC2: ACS758, alexmod:CB-PFF, F.Cu at (28.0, 122.0)
- added Q10: ZXTC2045E6, TO_SOT_Packages_SMD:SOT-23-6, F.Cu at (136.6, 141.0)
- added Q11: Q_NMOS_GDS, alexmod:TO-264_flat_reverse, B.Cu at (116.0, 106.8)
- added Q12: Q_NMOS_GDS, alexmod:TO-264_flat_reverse, B.Cu at (116.0, 137.2)
- added Q13: Q_NMOS_GDS, alexmod:TO-264_flat_reverse, B.Cu at (136.0, 106.8)
- added Q14: Q_NMOS_GDS, alexmod:TO-264_flat_reverse, B.Cu at (136.0, 137.2)
- added Q15: Q_NMOS_GDS, alexmod:TO-264_flat_reverse, B.Cu at (156.0, 106.8)
- added Q16: Q_NMOS_GDS, alexmod:TO-264_flat_reverse, B.Cu at (156.0, 137.2)
- added Q17: ZXTC2045E6, TO_SOT_Packages_SMD:SOT-23-6, F.Cu at (196.0, 98.4)
- added Q18: ZXTC2045E6, TO_SOT_Packages_SMD:SOT-23-6, F.Cu at (196.0, 141.3)
- added Q19: Q_NMOS_GDS, alexmod:TO-264_flat_reverse, B.Cu at (176.0, 106.8)
- added Q20: Q_NMOS_GDS, alexmod:TO-264_flat_reverse, B.Cu at (176.0, 137.2)
- added Q21: Q_NMOS_GDS, alexmod:TO-264_flat_reverse, B.Cu at (196.0, 106.8)
- added Q22: Q_NMOS_GDS, alexmod:TO-264_flat_reverse, B.Cu at (196.0, 137.2)
- added Q23: Q_NMOS_GDS, alexmod:TO-264_flat_reverse, B.Cu at (216.0, 106.8)
- added Q24: Q_NMOS_GDS, alexmod:TO-264_flat_reverse, B.Cu at (216.0, 137.2)
- added Q7: Q_NMOS_GDS, alexmod:TO-264_flat_reverse, B.Cu at (76.0, 106.8)
- added Q8: ZXTC2045E6, TO_SOT_Packages_SMD:SOT-23-6, F.Cu at (135.8, 98.4)
- added Q9: Q_NMOS_GDS, alexmod:TO-264_flat_reverse, B.Cu at (96.0, 137.2)
- added R14: 4R7, Resistors_SMD:R_0805, F.Cu at (101.5, 137.0)
- added R15: 120R, Resistors_SMD:R_0805, F.Cu at (134.8, 95.2)
- added R16: 120R, Resistors_SMD:R_0805, F.Cu at (133.5, 140.0)
- added R31: 10k, Resistors_SMD:R_0805, F.Cu at (201.4, 107.0)
- added R39: 4R7, Resistors_SMD:R_0805, F.Cu at (201.5, 137.0)
- added R40: 4R7, Resistors_SMD:R_0805, F.Cu at (221.5, 137.0)
- added R41: R, Resistors_SMD:R_0805, F.Cu at (65.4, 20.0)
- added REF**: MountingHole_3.2mm_M3, Mounting_Holes:MountingHole_3.2mm_M3, F.Cu at (99.2, 120.8)
- added REF**: MountingHole_3.2mm_M3, Mounting_Holes:MountingHole_3.2mm_M3, F.Cu at (99.2, 26.8)
- added REF**: MountingHole_3.2mm_M3, Mounting_Holes:MountingHole_3.2mm_M3, F.Cu at (172.8, 120.8)
- added REF**: MountingHole_3.2mm_M3, Mounting_Holes:MountingHole_3.2mm_M3, F.Cu at (172.8, 26.8)
- C1, C8: value 10u,50V -> 1u; footprint CRF1:SMD-1206 -> Capacitors_SMD:C_0805
- C10, C11, C12, C13: value 2.2u -> 100n; footprint CRF1:SMD-0603_c -> Capacitors_SMD:C_0805
- C14: value 2.2u -> 100n; footprint CRF1:SMD-0603_c -> Capacitors_SMD:C_0805; moved to F.Cu
- C2, C3: value 100n -> 1u; footprint CRF1:SMD-0603_c -> Capacitors_SMD:C_0805; moved to F.Cu
- C4, C5, C6, C7: value 4n7 -> 1u; footprint CRF1:SMD-0603_c -> Capacitors_SMD:C_0805; moved to F.Cu
- C41: value 2.2u -> 1u; footprint CRF1:SMD-0603_c -> Capacitors_SMD:C_0805
- C9: value 10u,50V -> 100n; footprint CRF1:SMD-1206 -> Capacitors_SMD:C_0805; moved to F.Cu
- D1: value GREEN -> RFN2L4S; footprint LEDs:LED-0603 -> Diodes_SMD:SMA_Standard; moved to F.Cu
- D2: value RED -> RFN2L4S; footprint LEDs:LED-0603 -> Diodes_SMD:SMA_Standard; moved to F.Cu
- D3: value LED -> RFN2L4S; footprint LEDs:LED-0603 -> Diodes_SMD:SMA_Standard; moved to F.Cu
- P1: value HALL/Encoder -> CONN_02X20; footprint CRF1:MICRO_JST_6 -> alexmod:XG4A_40
- P4, P5: footprint CRF1:1PAD_4x5mm -> Mounting_Holes:MountingHole_6.5mm_Pad_Via; moved to F.Cu
- P6, P7, P9: footprint CRF1:1PAD_4x5mm -> Mounting_Holes:MountingHole_6.5mm_Pad_Via
- Q1: value IRFS7530 -> ZXTC2045E6; footprint CRF1:D2PAK-7-GDS -> TO_SOT_Packages_SMD:SOT-23-6
- Q2: value IRFS7530 -> ZXTC2045E6; footprint CRF1:D2PAK-7-GDS -> TO_SOT_Packages_SMD:SOT-23-6; moved to F.Cu
- Q3, Q5: value IRFS7530 -> Q_NMOS_GDS; footprint CRF1:D2PAK-7-GDS -> alexmod:TO-264_flat_reverse; moved to B.Cu
- Q4, Q6: value IRFS7530 -> Q_NMOS_GDS; footprint CRF1:D2PAK-7-GDS -> alexmod:TO-264_flat_reverse
- R1: footprint CRF1:SMD-0603_r -> Resistors_SMD:R_0603
- R10, R9: value 10k -> 4R7; footprint CRF1:SMD-0603_r -> Resistors_SMD:R_0805; moved to F.Cu
- R11, R12, R13, R22: value 2k2 -> 4R7; footprint CRF1:SMD-0603_r -> Resistors_SMD:R_0805; moved to F.Cu
- R17: value 18k -> 10k; footprint CRF1:SMD-0603_r -> Resistors_SMD:R_0805
- R18: value 3k3 -> 10k; footprint CRF1:SMD-0603_r -> Resistors_SMD:R_0805
- R19: value 15k -> 4R7; footprint CRF1:SMD-0603_r -> Resistors_SMD:R_0805
- R2, R28: footprint CRF1:SMD-0603_r -> Resistors_SMD:R_0805
- R20: value 10k -> 4R7; footprint CRF1:SMD-0603_r -> Resistors_SMD:R_0805
- R21: value 220k -> 4R7; footprint CRF1:SMD-0603_r -> Resistors_SMD:R_0805; moved to F.Cu
- R23, R26, R3, R32: value 39k -> 64k9; footprint CRF1:SMD-0603_r -> Resistors_SMD:R_0805; moved to F.Cu
- R24, R27, R33, R4: value 2k2 -> 1k; footprint CRF1:SMD-0603_r -> Resistors_SMD:R_0805; moved to F.Cu
- R25: value 1M -> 4R7; footprint CRF1:SMD-0603_r -> Resistors_SMD:R_0805
- R29: value 4R7 -> 120R; footprint CRF1:SMD-0603_r -> Resistors_SMD:R_0805; moved to F.Cu
- R30: value 39k -> 120R; footprint CRF1:SMD-0603_r -> Resistors_SMD:R_0805; moved to F.Cu
- R34: value 4R7 -> 10k; footprint CRF1:SMD-0603_r -> Resistors_SMD:R_0805
- R35, R8: footprint CRF1:SMD-0603_r -> Resistors_SMD:R_0805; moved to F.Cu
- R36: value 39k -> 4R7; footprint CRF1:SMD-0603_r -> Resistors_SMD:R_0805; moved to F.Cu
- R37, R38: value 100R -> 4R7; footprint CRF1:SMD-0603_r -> Resistors_SMD:R_0805; moved to F.Cu
- R5: value 2k2 -> 10k; footprint CRF1:SMD-0603_r -> Resistors_SMD:R_0805; moved to F.Cu
- R6: value 0R -> 120R; footprint CRF1:SMD-0603_r -> Resistors_SMD:R_0805; moved to F.Cu
- R7: value 10k -> 120R; footprint CRF1:SMD-0603_r -> Resistors_SMD:R_0805; moved to F.Cu
- U1: value STM32F40X_LQFP64 -> IR2110S; footprint CRF1:lqfp64_pad_mod -> Housings_SOIC:SOIC-16_7.5x10.3mm_Pitch1.27mm
- U2: value TC2117 -> IR2110S; footprint CRF1:SOT-223 -> Housings_SOIC:SOIC-16_7.5x10.3mm_Pitch1.27mm; moved to F.Cu
- U3: value DRV8302 -> IR2110S; footprint CRF1:TSSOP-56-PP -> Housings_SOIC:SOIC-16_7.5x10.3mm_Pitch1.27mm
- moved R26 321.4 mm to (-233.1, 120.2)
- moved R27 301.6 mm to (-208.8, 120.2), turned to 0 degrees
- moved C14 290.0 mm to (-193.1, 101.8), turned to 0 degrees
- moved R33 277.3 mm to (-184.6, 120.2), turned to 0 degrees
- moved R4 222.0 mm to (-132.8, 87.2), turned to 0 degrees
- moved R24 216.7 mm to (-119.4, 83.4), turned to 0 degrees
- moved R23 200.2 mm to (-111.7, 120.2)
- moved R3 183.0 mm to (-92.8, 83.4), turned to 0 degrees
- moved R32 163.7 mm to (-75.3, 120.2)
- moved C1 120.0 mm to (216.5, 122.0), turned to 270 degrees
- moved P1 117.8 mm to (136.0, 30.0), turned to 180 degrees
- moved P6 117.6 mm to (196.0, 122.0), turned to 0 degrees
- moved C7 113.7 mm to (196.0, 101.6), turned to 0 degrees
- moved C8 108.3 mm to (199.0, 141.3), turned to 90 degrees
- moved R37 100.2 mm to (210.5, 107.0), turned to 90 degrees
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Connections:
- C1 pad 1: GND -> +3V3
- C1 pad 2: V_SUPPLY -> GND
- C10 pad 2: VCC -> +3V3
- C11 pad 2: VCC -> +3V3
- C12 pad 1: GND -> /Mosfet driver/H1_HI
- C12 pad 2: VCC -> /Mosfet driver/H1_VS
- C13 pad 1: GND -> /Mosfet driver/H2_HI
- C13 pad 2: VCC -> /Mosfet driver/H2_VS
- C14 pad 1: GND -> /Mosfet driver/H3_HI
- C14 pad 2: VCC -> /Mosfet driver/H3_VS
- C2 pad 1: GND -> +3V3
- C2 pad 2: /MCU/AN_IN -> GND
- C3 pad 1: GND -> /Mosfet driver/H1_HI
- C3 pad 2: /MCU/SERVO -> /Mosfet driver/H1_VS
- C4 pad 1: GND -> +12V
- C4 pad 2: /Filters/TEMP_IN -> /Mosfet driver/H1_LOW
- C41 pad 1: /MCU/ADC_TEMP -> /NTC temp sensor/Temp
- C5 pad 1: /Filters/HALL3_OUT -> /Mosfet driver/H2_HI
- C5 pad 2: GND -> /Mosfet driver/H2_VS
- C6 pad 1: /Filters/HALL2_OUT -> +12V
- C6 pad 2: GND -> GNDPWR
- C7 pad 1: /Filters/HALL1_OUT -> /Mosfet driver/H3_HI
- C7 pad 2: GND -> /Mosfet driver/H3_VS
- C8 pad 1: GND -> +12V
- C8 pad 2: V_SUPPLY -> /Mosfet driver/H3_LOW
- C9 pad 2: V_SUPPLY -> +3V3
- D1 pad 1: Net-(D1-Pad1) -> /Mosfet driver/H1_HI
- D1 pad 2: GND -> +12V
- D2 pad 1: Net-(D2-Pad1) -> /Mosfet driver/H2_HI
- D2 pad 2: GND -> +12V
- D3 pad 1: Net-(D3-Pad1) -> /Mosfet driver/H3_HI
- D3 pad 2: GND -> +12V
- P1 pad 1: +5V -> GND
- P1 pad 2: /Filters/TEMP_IN -> /Mosfet driver/EN_GATE
- P1 pad 3: /Filters/HALL1_IN -> GND
- P1 pad 4: /Filters/HALL2_IN -> /Mosfet driver/H1
- P1 pad 5: /Filters/HALL3_IN -> GND
- P1 pad 6: GND -> /Mosfet driver/L1
- P4 pad 1: V_SUPPLY -> +BATT
- P5 pad 1: GND -> GNDPWR
- R1 pad 1: VCC -> +3V3
- R1 pad 2: /MCU/ADC_TEMP -> /NTC temp sensor/Temp
- R10 pad 1: /Filters/HALL3_IN -> Net-(Q5-Pad1)
- R10 pad 2: /Filters/HALL3_OUT -> Net-(Q1-Pad4)
- R11 pad 1: /Filters/HALL3_IN -> Net-(Q7-Pad1)
- R11 pad 2: VCC -> Net-(Q1-Pad4)
- R12 pad 1: /Filters/HALL2_IN -> Net-(Q4-Pad1)
- R12 pad 2: VCC -> Net-(Q2-Pad4)
- R13 pad 1: /Filters/HALL1_IN -> Net-(Q6-Pad1)
- R13 pad 2: VCC -> Net-(Q2-Pad4)
- R17 pad 1: +5V -> /Mosfet driver/H2_VS
- R17 pad 2: Net-(R17-Pad2) -> Net-(Q8-Pad4)
- R18 pad 1: Net-(R17-Pad2) -> GNDPWR
- R18 pad 2: GND -> Net-(Q10-Pad4)
- R19 pad 2: Net-(C19-Pad2) -> Net-(Q8-Pad4)
- R2 pad 1: /MCU/ADC_TEMP -> /NTC temp sensor/Temp
- R20 pad 1: Net-(R20-Pad1) -> Net-(Q13-Pad1)
- R20 pad 2: GND -> Net-(Q8-Pad4)
- R21 pad 1: GND -> Net-(Q15-Pad1)
- R21 pad 2: Net-(R21-Pad2) -> Net-(Q8-Pad4)
- R22 pad 1: Net-(D3-Pad1) -> Net-(Q12-Pad1)
- R22 pad 2: VCC -> Net-(Q10-Pad4)
- R23 pad 2: /MCU/SENS1 -> /Mosfet driver/SENS1
- R24 pad 2: /MCU/SENS1 -> /Mosfet driver/SENS1
- R25 pad 1: GND -> Net-(Q14-Pad1)
- R25 pad 2: Net-(R25-Pad2) -> Net-(Q10-Pad4)
- R26 pad 2: /MCU/SENS2 -> /Mosfet driver/SENS2
- R27 pad 2: /MCU/SENS2 -> /Mosfet driver/SENS2
- R28 pad 1: Net-(Q1-PadG) -> Net-(Q16-Pad1)
- R28 pad 2: /Mosfet driver/M_H1 -> Net-(Q10-Pad4)
- R29 pad 1: Net-(Q2-PadG) -> /Mosfet driver/M_H3
- R29 pad 2: /Mosfet driver/M_L1 -> Net-(Q17-Pad4)
- R3 pad 1: V_SUPPLY -> +BATT
- R3 pad 2: /MCU/AN_IN -> Net-(P1-Pad28)
- R30 pad 1: /Mosfet driver/H1_LOW -> /Mosfet driver/M_L3
- R30 pad 2: Net-(Q2-PadG) -> Net-(Q18-Pad4)
- R32 pad 2: /MCU/SENS3 -> /Mosfet driver/SENS3
- R33 pad 2: /MCU/SENS3 -> /Mosfet driver/SENS3
- R34 pad 1: Net-(Q3-PadG) -> /Mosfet driver/H3_LOW
- R34 pad 2: /Mosfet driver/M_H2 -> Net-(Q18-Pad4)
- R35 pad 1: Net-(Q4-PadG) -> Net-(Q19-Pad1)
- R35 pad 2: /Mosfet driver/M_L2 -> Net-(Q17-Pad4)
- R36 pad 1: /Mosfet driver/H1_LOW -> Net-(Q21-Pad1)
- R36 pad 2: Net-(Q4-PadG) -> Net-(Q17-Pad4)
- R37 pad 1: Net-(D1-Pad1) -> Net-(Q23-Pad1)
- R37 pad 2: /MCU/LED_GREEN -> Net-(Q17-Pad4)
- R38 pad 1: Net-(D2-Pad1) -> Net-(Q20-Pad1)
- R38 pad 2: /MCU/LED_RED -> Net-(Q18-Pad4)
- R4 pad 1: GND -> Net-(P1-Pad28)
- R4 pad 2: /MCU/AN_IN -> GND
- R5 pad 1: /MCU/SERVO -> /Mosfet driver/H1_VS
- R5 pad 2: Net-(K1-Pad1) -> Net-(Q1-Pad4)
- R6 pad 1: Net-(R6-Pad1) -> /Mosfet driver/M_H1
- R6 pad 2: +5V -> Net-(Q1-Pad4)
- R7 pad 1: /Filters/TEMP_IN -> /Mosfet driver/M_L1
- R7 pad 2: VCC -> Net-(Q2-Pad4)
- R8 pad 1: /Filters/HALL1_IN -> /Mosfet driver/H1_LOW
- R8 pad 2: /Filters/HALL1_OUT -> Net-(Q2-Pad4)
- R9 pad 1: /Filters/HALL2_IN -> Net-(Q3-Pad1)
- R9 pad 2: /Filters/HALL2_OUT -> Net-(Q1-Pad4)
- U1 pad 1: VCC -> /Mosfet driver/M_L1
- U1 pad 10: /MCU/AN_IN -> (no net)
- U1 pad 11: Net-(U1-Pad11) -> +3V3
- U1 pad 12: GND -> /Mosfet driver/H1
- U1 pad 13: VCC -> /Mosfet driver/EN_GATE
- U1 pad 14: /MCU/SENS3 -> /Mosfet driver/L1
- U1 pad 15: /MCU/SENS2 -> GND
- U1 pad 16: /MCU/SENS1 -> (no net)
- U1 pad 2: Net-(U1-Pad2) -> /Mosfet driver/H1_LOW
- U1 pad 3: Net-(U1-Pad3) -> +12V
- U1 pad 4: Net-(U1-Pad4) -> (no net)
- U1 pad 5: Net-(C15-Pad1) -> (no net)
- U1 pad 6: Net-(C38-Pad1) -> /Mosfet driver/H1_VS
- U1 pad 7: NRST -> /Mosfet driver/H1_HI
- U1 pad 8: /Filters/TEMP_IN -> /Mosfet driver/M_H1
- U1 pad 9: Net-(U1-Pad9) -> (no net)
- U2 pad 1: GND -> /Mosfet driver/M_L2
- U2 pad 2: VCC -> GNDPWR
- U2 pad 3: +5V -> +12V
- U3 pad 1: Net-(R21-Pad2) -> /Mosfet driver/M_L3
- U3 pad 10: GND -> (no net)
- U3 pad 11: Net-(C20-Pad2) -> +3V3
- U3 pad 12: /MCU/DC_CAL -> /Mosfet driver/H3
- U3 pad 13: Net-(C18-Pad1) -> /Mosfet driver/EN_GATE
- U3 pad 14: Net-(C22-Pad1) -> /Mosfet driver/L3
- U3 pad 15: Net-(C22-Pad2) -> GND
- U3 pad 16: /MCU/EN_GATE -> (no net)
- U3 pad 2: Net-(C19-Pad2) -> /Mosfet driver/H3_LOW
- U3 pad 3: Net-(R17-Pad2) -> +12V
- U3 pad 4: Net-(U3-Pad4) -> (no net)
- U3 pad 5: Net-(U3-Pad5) -> (no net)
- U3 pad 6: /MCU/FAULT -> /Mosfet driver/H3_VS
- U3 pad 7: Net-(R20-Pad1) -> /Mosfet driver/H3_HI
- U3 pad 8: GND -> /Mosfet driver/M_H3
- U3 pad 9: VCC -> (no net)
Routing:
- net +12V: track 0.00 -> 728.1 mm, vias 0 -> 1
- net GND: track 398.8 -> 12.7 mm, vias 27 -> 0
- net /Mosfet driver/H3_LOW: track 53.5 -> 392.5 mm, vias 2 -> 0
- net GNDPWR: track 0.00 -> 315.2 mm
- net /Mosfet driver/M_L3: track 20.0 -> 316.3 mm, vias 2 -> 0
- net V_SUPPLY: track 290.3 -> 0.00 mm, vias 20 -> 0
- net +BATT: track 0.00 -> 272.1 mm
- net +3V3: track 0.00 -> 269.3 mm, vias 0 -> 1
- net /Mosfet driver/M_L2: track 19.3 -> 234.8 mm, vias 2 -> 0
- net VCC: track 185.2 -> 0.00 mm, vias 9 -> 0
- net /Mosfet driver/H1_LOW: track 48.5 -> 219.9 mm, vias 2 -> 0
- net Net-(IC1-Pad2): track 0.00 -> 163.7 mm, vias 0 -> 1
- net /Mosfet driver/H3_HI: track 0.00 -> 137.3 mm
- net +5V: track 115.3 -> 0.00 mm, vias 4 -> 0
- net /Mosfet driver/M_L1: track 28.9 -> 134.0 mm, vias 2 -> 0
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- added copper zone on B.Cu, net +BATT
- added copper zone on B.Cu, net GNDPWR
- removed copper zone on GND, net /Mosfet driver/H1_VS
- removed copper zone on GND2, net /Mosfet driver/H1_VS
- removed copper zone on GND, net /Mosfet driver/H2_VS
- removed copper zone on GND2, net /Mosfet driver/H2_VS
- removed copper zone on GND, net /Mosfet driver/H3_VS
- removed copper zone on GND2, net /Mosfet driver/H3_VS
- removed copper zone on B.Cu, net GND
- removed copper zone on F.Cu, net GND
- removed copper zone on GND, net GND
- removed copper zone on GND2, net GND
- removed copper zone on B.Cu, net VCC
- removed copper zone on F.Cu, net V_SUPPLY
Other:
- board outline removed
- copper layers 4 -> 2
- net class Default: clearance 0.1778 -> 0.3; trace_width 0.2032 -> 0.4; via_dia 0.8 -> 1.8; via_drill 0.5 -> 0.9
- rule trace_clearance: 0.1778 -> 0.3
- rule trace_min: 0.2032 -> 0.2
- rule via_min_drill: 0.5 -> 0.3
- rule via_min_size: 0.8 -> 0.4
- board text removed: "3.3V"
- board text removed: "3.3v"
- board text removed: "5v"
- board text removed: "ADC"
- board text removed: "ADC2"
- board text removed: "Benjamin Vedder"
- board text removed: "CANH"
- board text removed: "CANL"
- board text removed: "CLK"
- board text removed: "DIO"
- board text removed: "GND"
- board text removed: "H1"
- board text removed: "H2"
- board text removed: "H3"
- board text removed: "MISO"
- board text removed: "MOSI"
- board text removed: "NSS"
- board text removed: "RST"
- board text removed: "RX"
- board text removed: "SCK"
- board text removed: "SCL"
- board text removed: "SDA"
- board text removed: "TEMP"
- board text removed: "TX"
- board text removed: "VESC 4.12"
- board text removed: "vedder.se"
