File: board/BLDC_4.kicad_pcb (KiCad board)
At the start: 2 copper layers, 98 parts, among them IC1 ACS758, IC2 ACS758, P1 CONN_02X20, P4 IN+, P5 IN-, P6 MOTOR1, P7 MOTOR2, P9 MOTOR3, Q1 ZXTC2045E6, Q10 ZXTC2045E6, Q11 Q_NMOS_GDS, Q12 Q_NMOS_GDS, Q13 Q_NMOS_GDS, Q14 Q_NMOS_GDS, Q15 Q_NMOS_GDS, Q16 Q_NMOS_GDS, Q17 ZXTC2045E6, Q18 ZXTC2045E6, Q19 Q_NMOS_GDS, Q2 ZXTC2045E6, Q20 Q_NMOS_GDS, Q21 Q_NMOS_GDS, Q22 Q_NMOS_GDS, Q23 Q_NMOS_GDS, Q24 Q_NMOS_GDS, Q3 Q_NMOS_GDS, Q4 Q_NMOS_GDS, Q5 Q_NMOS_GDS, Q6 Q_NMOS_GDS, Q7 Q_NMOS_GDS, Q8 ZXTC2045E6, Q9 Q_NMOS_GDS, U1 IR2110S, U2 IR2110S, U3 IR2110S

Commit message: - preliminary finish of layout
Parts:
- R41: moved to B.Cu
- moved C14 432.6 mm to (238.2, 68.8), turned to 180 degrees
- moved R26 403.5 mm to (163.2, 44.2), turned to 90 degrees
- moved R27 380.4 mm to (163.2, 41.0), turned to 270 degrees
- moved R33 358.6 mm to (165.2, 41.0), turned to 270 degrees
- moved R23 346.1 mm to (230.0, 65.6), turned to 180 degrees
- moved R32 302.1 mm to (221.2, 62.6)
- moved R4 297.6 mm to (161.2, 41.0), turned to 90 degrees
- moved R24 289.7 mm to (167.2, 41.0), turned to 270 degrees
- moved R3 227.3 mm to (132.6, 54.0), turned to 90 degrees
- moved C10 151.3 mm to (225.0, 46.4)
- moved C11 151.3 mm to (238.0, 46.4)
- moved C12 151.3 mm to (212.2, 69.6)
- moved C13 151.3 mm to (225.2, 69.6)
- moved C9 151.3 mm to (212.0, 46.4)
- moved D1 151.3 mm to (211.2, 65.4)
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Routing:
- net GND: track 12.7 -> 577.0 mm, vias 0 -> 6
- net GNDPWR: track 315.2 -> 93.5 mm, vias 0 -> 2
- net +12V: track 728.1 -> 925.5 mm, vias 1 -> 3
- net Net-(IC2-Pad2): track 3.93 -> 184.1 mm
- net /NTC temp sensor/Temp: track 7.32 -> 173.2 mm
- net +3V3: track 269.3 -> 433.2 mm
- net /Mosfet driver/EN_GATE: track 4.34 -> 152.8 mm, vias 1 -> 3
- net /Mosfet driver/H3_LOW: track 392.5 -> 249.3 mm, vias 0 -> 1
- net /Mosfet driver/M_L1: track 134.0 -> 273.9 mm
- net /Mosfet driver/H1_LOW: track 219.9 -> 359.7 mm, vias 0 -> 1
- net /Mosfet driver/H1_VS: track 87.0 -> 223.3 mm
- net /Mosfet driver/M_L3: track 316.3 -> 183.1 mm
- net /Mosfet driver/H2_VS: track 105.3 -> 235.9 mm
- net /Mosfet driver/M_H1: track 56.6 -> 174.6 mm
- net /Mosfet driver/H1_HI: track 56.2 -> 171.2 mm
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
Commit message: - added mounting holes - added local zero - added outline
Parts:
- added REF**: MountingHole_3.2mm_M3, Mounting_Holes:MountingHole_3.2mm_M3, F.Cu at (25.0, 20.0)
- added REF**: MountingHole_3.2mm_M3, Mounting_Holes:MountingHole_3.2mm_M3, F.Cu at (25.0, 162.0)
- added REF**: MountingHole_3.2mm_M3, Mounting_Holes:MountingHole_3.2mm_M3, F.Cu at (257.0, 162.0)
- added REF**: MountingHole_3.2mm_M3, Mounting_Holes:MountingHole_3.2mm_M3, F.Cu at (257.0, 20.0)
Other:
- board outline added: 240 x 150 mm
Changed lines of the file:
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@@
 (kicad_pcb (version 4) (host pcbnew 4.0.0-rc1-stable)
   (general
-    (links 235)
-    (no_connects 25)
-    (area 0 0 0 0)
+    (links 0)
+    (no_connects 19)
+    (area 23.774999 20.899999 260.000001 164.775001)
     (thickness 1.6)
-    (drawings 0)
+    (drawings 4)
     (tracks 840)
     (zones 0)
-    (modules 98)
+    (modules 102)
     (nets 58)
   )
@@
     (add_net "Net-(Q9-Pad1)")
   )
+  (module Mounting_Holes:MountingHole_3.2mm_M3 (layer F.Cu)
+    (at 25 20)
+    (descr "Mounting Hole 3.2mm, no annular, M3")
+    (tags "mounting hole 3.2mm no annular m3")
+    (fp_text reference REF** (at 0 -4.2) (layer F.SilkS)
+      (effects (font (size 1 1) (thickness 0.15)))
+    )
+    (fp_text value MountingHole_3.2mm_M3 (at 0 4.2) (layer F.Fab)
+      (effects (font (size 1 1) (thickness 0.15)))
+    )
+    (fp_circle (center 0 0) (end 3.2 0) (layer Cmts.User) (width 0.15))
+    (fp_circle (center 0 0) (end 3.45 0) (layer F.CrtYd) (width 0.05))
+    (pad 1 np_thru_hole circle (at 0 0) (size 3.2 3.2) (drill 3.2) (layers *.Cu *.Mask F.SilkS))
+  )
+  (module Mounting_Holes:MountingHole_3.2mm_M3 (layer F.Cu)
+    (at 25 162)
+    (descr "Mounting Hole 3.2mm, no annular, M3")
+    (tags "mounting hole 3.2mm no annular m3")
+    (fp_text reference REF** (at 0 -4.2) (layer F.SilkS)
+      (effects (font (size 1 1) (thickness 0.15)))
+    )
+    (fp_text value MountingHole_3.2mm_M3 (at 0 4.2) (layer F.Fab)
+      (effects (font (size 1 1) (thickness 0.15)))
+    )
+    (fp_circle (center 0 0) (end 3.2 0) (layer Cmts.User) (width 0.15))
+    (fp_circle (center 0 0) (end 3.45 0) (layer F.CrtYd) (width 0.05))
+    (pad 1 np_thru_hole circle (at 0 0) (size 3.2 3.2) (drill 3.2) (layers *.Cu *.Mask F.SilkS))
+  )
+  (module Mounting_Holes:MountingHole_3.2mm_M3 (layer F.Cu)
+    (at 257 162)
+    (descr "Mounting Hole 3.2mm, no annular, M3")
+    (tags "mounting hole 3.2mm no annular m3")
+    (fp_text reference REF** (at 0 -4.2) (layer F.SilkS)
+      (effects (font (size 1 1) (thickness 0.15)))
+    )
+    (fp_text value MountingHole_3.2mm_M3 (at 0 4.2) (layer F.Fab)
+      (effects (font (size 1 1) (thickness 0.15)))
+    )
+    (fp_circle (center 0 0) (end 3.2 0) (layer Cmts.User) (width 0.15))
+    (fp_circle (center 0 0) (end 3.45 0) (layer F.CrtYd) (width 0.05))
+    (pad 1 np_thru_hole circle (at 0 0) (size 3.2 3.2) (drill 3.2) (layers *.Cu *.Mask F.SilkS))
+  )
   (module Housings_SOIC:SOIC-16_7.5x10.3mm_Pitch1.27mm (layer F.Cu)
     (at 223.2 55.4 90)
@@
       (net 48 "Net-(Q14-Pad1)"))
   )
+  (module Mounting_Holes:MountingHole_3.2mm_M3 (layer F.Cu)
+    (at 257 20)
+    (descr "Mounting Hole 3.2mm, no annular, M3")
+    (tags "mounting hole 3.2mm no annular m3")
+    (fp_text reference REF** (at 0 -4.2) (layer F.SilkS)
+      (effects (font (size 1 1) (thickness 0.15)))
+    )
+    (fp_text value MountingHole_3.2mm_M3 (at 0 4.2) (layer F.Fab)
+      (effects (font (size 1 1) (thickness 0.15)))
+    )
+    (fp_circle (center 0 0) (end 3.2 0) (layer Cmts.User) (width 0.15))
+    (fp_circle (center 0 0) (end 3.45 0) (layer F.CrtYd) (width 0.05))
+    (pad 1 np_thru_hole circle (at 0 0) (size 3.2 3.2) (drill 3.2) (layers *.Cu *.Mask F.SilkS))
+  )
+  (gr_line (start 21 166) (end 261 166) (layer Edge.Cuts) (width 0.15))
+  (gr_line (start 21 16) (end 21 166) (layer Edge.Cuts) (width 0.15))
+  (gr_line (start 261 16) (end 21 16) (layer Edge.Cuts) (width 0.15))
+  (gr_line (start 261 166) (end 261 16) (layer Edge.Cuts) (width 0.15))
   (segment (start 225 99.35) (end 246.191169 99.35) (width 0.4) (layer F.Cu) (net 1))
   (segment (start 246.191169 99.35) (end 246.191169 78.917056) (width 0.4) (layer F.Cu) (net 1))
